Commit message: Add Franka Hand control with a shared sim/real interface
- Enable the Franka Hand in the Gazebo URDF (finger_joint2 as state-only mimic)
- Add fr3_gripper_controller (JointGroupPositionController)
- New aided_building_gripper package: sim server exposing the franka_gripper
  actions (homing, move, grasp, gripper_action, stop) and a CLI test tool
- Pin franka_description to 2.9.0 and add franka_ros2 (jazzy)

Co-Authored-By: Claude Opus 5.5 <noreply@anthropic.com>
Claude-Session: https://claude.ai/code/session_017hyrdbDad13F1RrDuQqbLW

File: aided_building_ws/src/aided_building_description/urdf/franka_gazebo.urdf.xacro (robot description, xacro)
@@ -4,5 +4,5 @@
   <xacro:arg name="rpy" default="0 0 0"/>
   <xacro:arg name="connected_to" default=""/>
-  <xacro:arg name="hand" default="false"/>
+  <xacro:arg name="hand" default="true"/>
   <xacro:arg name="include_self_collision_geometry" default="false"/>
   <link name="world"/>
@@ -66,4 +66,20 @@
       <state_interface name="velocity"/>
     </joint>
+    <!-- Franka Hand: only finger_joint1 is commanded (finger position = width / 2).
+         finger_joint2 is a URDF mimic joint; it must be listed here with state
+         interfaces only, otherwise gz_ros2_control does not drive it. -->
+    <joint name="fr3_finger_joint1">
+      <command_interface name="position"/>
+      <state_interface name="position">
+        <param name="initial_value">0.04</param>
+      </state_interface>
+      <state_interface name="velocity"/>
+    </joint>
+    <joint name="fr3_finger_joint2">
+      <state_interface name="position">
+        <param name="initial_value">0.04</param>
+      </state_interface>
+      <state_interface name="velocity"/>
+    </joint>
   </ros2_control>
   <gazebo>
@@ -75,3 +91,22 @@
     </plugin>
   </gazebo>
+  <!-- Rubber finger pads (same values as the official franka_gazebo). -->
+  <gazebo reference="fr3_leftfinger">
+    <collision>
+      <max_contacts>10</max_contacts>
+      <surface>
+        <contact><ode><max_vel>0</max_vel><min_depth>0.001</min_depth></ode></contact>
+        <friction><ode><mu>1.13</mu><mu2>1.13</mu2></ode></friction>
+      </surface>
+    </collision>
+  </gazebo>
+  <gazebo reference="fr3_rightfinger">
+    <collision>
+      <max_contacts>10</max_contacts>
+      <surface>
+        <contact><ode><max_vel>0</max_vel><min_depth>0.001</min_depth></ode></contact>
+        <friction><ode><mu>1.13</mu><mu2>1.13</mu2></ode></friction>
+      </surface>
+    </collision>
+  </gazebo>
 </robot>
